Commit message: S:Added Gazebo launch file, diffdrive controller, fixed urdf base_footprint issue

File: description/robot.urdf.xacro (robot description, xacro)
@@ -2,3 +2,4 @@
 <robot xmlns:xacro="http://www.ros.org/wiki/xacro" name="robot" >
     <xacro:include filename="robot_core.xacro" />
+    <xacro:include filename="gazebo_control.xacro"/>
 </robot>

File: description/robot_core.xacro (robot description, xacro)
@@ -11,5 +11,4 @@
         <color rgba="0.7 0.7 0.7 1" />
     </material>
-    <link name="base_footprint" />
     <!-- BASE LINK -->
     <link name="base_link">
@@ -31,9 +30,7 @@
         </xacro:inertial_box>
     </link>
-    <joint name="base_joint" type="fixed">
-        <parent link="base_footprint" />
-        <child link="base_link" />
-        <origin xyz="0 0 0.1" rpy="0 0 0" />
-    </joint>
+    <gazebo reference="base_link">
+        <material>Gazebo/Green</material>
+    </gazebo>
     <!-- LIDAR LINK -->
     <link name="lidar_link">
@@ -60,4 +57,7 @@
         <origin xyz="0 0 0.225" rpy="0 0 0" />
     </joint>
+    <gazebo reference="lidar_link">
+        <material>Gazebo/Blue</material>
+    </gazebo>
     <!-- LEFT WHEEL LINK -->
     <link name="left_wheel_link">
@@ -85,4 +85,7 @@
         <axis xyz="0 1 0" />
     </joint>
+    <gazebo reference="left_wheel_link">
+        <material>Gazebo/Grey</material>
+    </gazebo>
     <!-- RIGHT WHEEL LINK -->
     <link name="right_wheel_link">
@@ -110,4 +113,7 @@
         <axis xyz="0 1 0" />
     </joint>
+    <gazebo reference="right_wheel_link">
+        <material>Gazebo/Grey</material>
+    </gazebo>
     <!-- CASTER WHEEL LINK -->
     <link name="caster_wheel_link">
@@ -134,3 +140,8 @@
         <origin xyz="0.2 0 0" rpy="0 0 0"/>
     </joint>
+    <gazebo reference="caster_wheel_link">
+        <material>Gazebo/Grey</material>
+        <mu1 value ="0.001"/>
+        <mu2 value ="0.001"/>
+    </gazebo>
 </robot>

Commit message: S:Added lidar.xacro; rviz2 and Gazebo can use LiDAR

File: description/robot.urdf.xacro (robot description, xacro)
@@ -3,3 +3,4 @@
     <xacro:include filename="robot_core.xacro" />
     <xacro:include filename="gazebo_control.xacro"/>
+    <xacro:include filename="lidar.xacro"/>
 </robot>

File: description/robot_core.xacro (robot description, xacro)
@@ -32,31 +32,4 @@
     <gazebo reference="base_link">
         <material>Gazebo/Green</material>
-    </gazebo>
-    <!-- LIDAR LINK -->
-    <link name="lidar_link">
-        <visual>
-            <geometry>
-                <cylinder radius="0.1" length="0.05" />
-            </geometry>
-            <origin xyz="0 0 0" rpy="0 0 0" />
-            <material name="blue" />
-        </visual>
-        <collision>
-            <geometry>
-                <cylinder radius="0.1" length="0.05" />
-            </geometry>
-            <origin xyz="0 0 0" rpy="0 0 0" />
-        </collision>
-        <xacro:inertial_cylinder mass="0.1" radius="0.1" length="0.05" >
-            <origin xyz="0 0 0" rpy="0 0 0" />
-        </xacro:inertial_cylinder>
-    </link>
-    <joint name="base_lidar_joint" type="fixed">
-        <parent link="base_link" />
-        <child link="lidar_link" />
-        <origin xyz="0 0 0.225" rpy="0 0 0" />
-    </joint>
-    <gazebo reference="lidar_link">
-        <material>Gazebo/Blue</material>
     </gazebo>
     <!-- LEFT WHEEL LINK -->
